File: pcbs/pcb_using_pico/psion-org2-bluetooth-adapter/file61D041BF.sch (KiCad schematic (older format))
At the start: 6 parts

Commit message: V1_0 PCB sent off
Parts:
- added M1: P-CHANNEL-MOSFET, Package_TO_SOT_SMD:SOT-23, symbol GeekAmmo:P-CHANNEL-MOSFET
- added R1, R2: R_Small, Resistor_SMD:R_0805_2012Metric, symbol Device:R_Small
- added TR1: New_Library_Si2302CDS-n-channel, Package_TO_SOT_SMD:SOT-23, symbol cq1re1-cache:New_Library_Si2302CDS-n-channel
- C3: renamed from C?; footprint Capacitor_SMD:C_0805_2012Metric -> Capacitor_SMD:C_1206_3216Metric_Pad1.42x1.75mm_HandSolder
- gave numbers to parts that had none: 5
Connections:
- net GND: now also R1.2, TR1.2 (S)
- net VCC_ESP: now also M1.3 (D)
- new net: M1.1 (G), R2.2, TR1.3 (D)
- new net +3V3: M1.2 (S), R2.1
- new net WROOM_ON: R1.1, TR1.1 (G)
Other:
- note added: "WROOM\nProgramming"
- moved on the sheet: C3, C4, J2, JP5, R6, U4

Commit message: Changed circuit to new power arrangement
Parts:
- R1, R2: value R_Small -> 10k
- R6: value R_Small -> 47k
Changed lines of the file:
@@
 encoding utf-8
 Sheet 2 3
-Title ""
-Date ""
-Rev ""
+Title "Psion Organiser Bluetooth Adapter"
+Date "2022-01-01"
+Rev "1.1"
 Comp ""
 Comment1 ""
@@
 AR Path="/61D041C0/61D1E6BC" Ref="R6"  Part="1"
 F 0 "R6" H 6859 1896 50  0000 L CNN
-F 1 "R_Small" H 6859 1805 50  0000 L CNN
+F 1 "47k" H 6859 1805 50  0000 L CNN
 F 2 "Resistor_SMD:R_0805_2012Metric" H 6800 1850 50  0001 C CNN
 F 3 "~" H 6800 1850 50  0001 C CNN
@@
 P 1950 1125
 F 0 "R2" H 2009 1171 50  0000 L CNN
-F 1 "R_Small" H 2009 1080 50  0000 L CNN
+F 1 "10k" H 2009 1080 50  0000 L CNN
 F 2 "Resistor_SMD:R_0805_2012Metric" H 1950 1125 50  0001 C CNN
 F 3 "~" H 1950 1125 50  0001 C CNN
@@
 P 1525 2575
 F 0 "R1" H 1584 2621 50  0000 L CNN
-F 1 "R_Small" H 1584 2530 50  0000 L CNN
+F 1 "10k" H 1584 2530 50  0000 L CNN
 F 2 "Resistor_SMD:R_0805_2012Metric" H 1525 2575 50  0001 C CNN
 F 3 "~" H 1525 2575 50  0001 C CNN
