File: pcbs/pcb_using_pico/psion-org2-bluetooth-adapter/psion-org2-bluetooth-adapter.sch (KiCad schematic (older format))
At the start: 15 parts, among them J1 Conn_02x08_Odd_Even, J5 Conn_01x04_Female, J7 Conn_01x03_Female, U1 74LS245, U2 74LS245, U3 Pico

Commit message: V1_0 PCB sent off
Parts:
- added D1: D_Schottky, Diode_SMD:D_SOD-123, symbol Device:D_Schottky
Connections:
- net at U3.39 (VSYS): now also D1.1 (K)
- net IO0: no longer names the net of U3.1 (GPIO0)
- net IO1: no longer names the net of U3.2 (GPIO1)
- net IO2 renamed WROOM_ON
- net IO3: no longer names the net of U3.21 (GPIO16)
- net IO7: no longer names the net of U3.31 (GPIO26_ADC0)
- new net VREG: D1.2 (A)
Other:
- note removed: "XC9110C\n18650\nMCP73831\nMIC5504\n"
Changed lines of the file:
@@
 $Descr A4 11693 8268
 encoding utf-8
-Sheet 1 2
+Sheet 1 3
 Title ""
 Date ""
@@
 Text GLabel 1425 1375 0    50   Input ~ 0
 VB
-Text GLabel 8500 2625 0    50   Input ~ 0
-IO0
-Text GLabel 8500 2725 0    50   Input ~ 0
-IO1
-Text GLabel 9900 4125 2    50   Input ~ 0
-IO2
-Text GLabel 9900 4525 2    50   Input ~ 0
-IO3
 Text GLabel 9900 3925 2    50   Input ~ 0
 IP_CLK
 Text GLabel 9900 3725 2    50   Input ~ 0
 OP_CLK
-Text GLabel 9900 3525 2    50   Input ~ 0
-IO7
-$Comp
-L power:GND #PWR?
+$Comp
+L power:GND #PWR0107
 U 1 1 61CED555
 P 2575 5025
-F 0 "#PWR?" H 2575 4775 50  0001 C CNN
+F 0 "#PWR0107" H 2575 4775 50  0001 C CNN
 F 1 "GND" H 2580 4852 50  0000 C CNN
 F 2 "" H 2575 5025 50  0001 C CNN
@@
 $EndComp
 $Comp
-L power:GND #PWR?
+L power:GND #PWR0108
 U 1 1 61CEDAFC
 P 3450 4725
-F 0 "#PWR?" H 3450 4475 50  0001 C CNN
+F 0 "#PWR0108" H 3450 4475 50  0001 C CNN
 F 1 "GND" H 3455 4552 50  0000 C CNN
 F 2 "" H 3450 4725 50  0001 C CNN
@@
 $EndComp
 $Comp
-L power:GND #PWR?
+L power:GND #PWR0113
 U 1 1 61CEDD65
 P 3675 7125
-F 0 "#PWR?" H 3675 6875 50  0001 C CNN
+F 0 "#PWR0113" H 3675 6875 50  0001 C CNN
 F 1 "GND" H 3680 6952 50  0000 C CNN
 F 2 "" H 3675 7125 50  0001 C CNN
@@
 $EndComp
 $Comp
-L power:GND #PWR?
+L power:GND #PWR0114
 U 1 1 61CEDF39
 P 6400 4025
-F 0 "#PWR?" H 6400 3775 50  0001 C CNN
+F 0 "#PWR0114" H 6400 3775 50  0001 C CNN
 F 1 "GND" H 6405 3852 50  0000 C CNN
 F 2 "" H 6400 4025 50  0001 C CNN
@@
 $EndComp
 $Comp
-L power:GND #PWR?
+L power:GND #PWR0115
 U 1 1 61CEE0B8
 P 9725 6150
-F 0 "#PWR?" H 9725 5900 50  0001 C CNN
+F 0 "#PWR0115" H 9725 5900 50  0001 C CNN
 F 1 "GND" H 9730 5977 50  0000 C CNN
 F 2 "" H 9725 6150 50  0001 C CNN
@@
 Text Notes 8025 2050 0    50   ~ 0
 Pico USB could be used as USB \nserial if a connection is made to it.
-Text Notes 5550 4950 0    50   ~ 0
-XC9110C\n18650\nMCP73831\nMIC5504\n
+Text GLabel 9900 4125 2    50   Input ~ 0
+WROOM_ON
+$Comp
+L Device:D_Schottky D1
+U 1 1 61D1AB6B
+P 10725 2200
+F 0 "D1" V 10771 2121 50  0000 R CNN
+F 1 "D_Schottky" V 10680 2121 50  0000 R CNN
+F 2 "Diode_SMD:D_SOD-123" H 10725 2200 50  0001 C CNN
+F 3 "~" H 10725 2200 50  0001 C CNN
+	1    10725 2200
+	0    -1   -1   0
+$EndComp
+Wire Wire Line
+	10725 2350 10725 2725
+Wire Wire Line
+	10725 2725 9900 2725
+Text GLabel 10525 1825 0    50   Input ~ 0
+VREG
+Wire Wire Line
+	10525 1825 10725 1825
+Wire Wire Line
+	10725 1825 10725 2050
+$Sheet
+S 4250 5025 1450 700
+U 61D0535C
+F0 "Sheet61D0535B" 50
+F1 "Power.sch" 50
+$EndSheet
 $EndSCHEMATC

Commit message: Added code
Parts:
- added R?: 10k, symbol Device:R_Small
- added R?: 100k, symbol Device:R_Small
- added TR?: Si2302CDS-n-channel, Package_TO_SOT_SMD:SOT-23, symbol New_Library:Si2302CDS-n-channel
Connections:
- net GND: now also R?.2, TR?.2 (S)
- net SD3: now also R?.2, TR?.3 (D)
- net VCC: now also R?.1
- net TX_TO_PSION: now reaches U3.24 (GPIO18)
- net TX_TO_PSION: now also R?.1, TR?.1 (G)
- net IP_CLK: no longer names the net of U3.27 (GPIO21)
- net OP_CLK: no longer names the net of U3.29 (GPIO22)
Other:
- note added: "Bluetooth Adapter Breakout Board\nAttaches to top slot and allows Bluetooth communication\nCan have ROM in Pico flash (COMMS link)\nRTS/DTS not used\nOLED display for debug only, not needed for final PCB\n"
- note added: "The 74LVC245 diection is set for all 8 data bits,\nso we run a separate TX from the Pico to the RX of the\nPsion (on bit 3). This is open collector as a level shifter\nand also inverts the data. Fortunately a stop bit is a 1 and a \nstart bit is a 0. The transistor being off can be driven by the psion\nwhen loading the ROM and is seen as a stop bit (idle) when in\nserial mode."
- note removed: "Top Slot Adapter Breakout Board\nAttaches to top slot and provides general hardware interface\nCan have ROM in Pico flash"
- moved on the sheet: J5, JP1, JP2, JP3, JP4, R4, R5

Commit message: Updates
Parts:
- added M?: GeekAmmo_P-CHANNEL-MOSFET, SOT23-3, symbol cq1re1-cache:GeekAmmo_P-CHANNEL-MOSFET
- added R?: 4k7, symbol Device:R_Small
- added R?: 10k, symbol Device:R_Small
- added TR?: Si2302CDS-n-channel, Package_TO_SOT_SMD:SOT-23, symbol New_Library:Si2302CDS-n-channel
- R?: value 100k -> 10k
Connections:
- net GND: now also R?.2, TR?.2 (S)
- net SD3: now also M?.3 (D); no longer R?.2
- net VCC: now also R?.1, R?.1; no longer R?.1
- net TRITX: now reaches U3.21 (GPIO16)
- net TRITX: now also R?.1, TR?.1 (G)
- new net: M?.1 (G), R?.2, TR?.3 (D)
- new net: M?.2 (S), R?.2
Other:
- moved on the sheet: C1, R?, TR?, U1
