File: pcbs/pcb_using_pico/psion-org2-bluetooth-adapter/p1.sch (KiCad schematic (older format))
At the start: 22 parts, among them J3 Barrel_Jack, J4 Connector_USB_B_Micro, U6 AMS1117-3.3, U7 AMS1117-5.0, U8 ETA6002

Commit message: Merged erroneous changes to V1.0 archive started
Parts:
- removed BT2: Battery_Cell, Battery:BatteryHolder_Keystone_1042_1x18650, symbol Device:Battery_Cell
- removed C13, C6: 100nF, Capacitor_SMD:C_0805_2012Metric, symbol Device:C_Small
- removed C15: 22uF, Capacitor_SMD:C_1206_3216Metric_Pad1.42x1.75mm_HandSolder, symbol Device:C_Small
- removed C16, C5: 10uF, Capacitor_SMD:C_1206_3216Metric_Pad1.42x1.75mm_HandSolder, symbol Device:C_Small
- removed C9: 1uF, Capacitor_SMD:C_1206_3216Metric_Pad1.42x1.75mm_HandSolder, symbol Device:C_Small
- removed D4: LED, LED_SMD:LED_0805_2012Metric_Pad1.15x1.40mm_HandSolder, symbol Device:LED
- removed J3: Barrel_Jack, Connector_BarrelJack:BarrelJack_Horizontal, symbol Connector:Barrel_Jack
- removed J4: Connector_USB_B_Micro, Connector_USB:USB_Micro-B_GCT_USB3076-30-A, symbol cq1re1-cache:Connector_USB_B_Micro
- removed JP6: Jumper_NO_Small, Jumper:SolderJumper-2_P1.3mm_Open_RoundedPad1.0x1.5mm, symbol Device:Jumper_NO_Small
- removed L1: 2.2uH, Inductor_SMD:L_Coilcraft_LPS5030, symbol Device:L
- removed R13: 2k2, Resistor_SMD:R_0805_2012Metric, symbol Device:R_Small
- removed R14: 500R, Resistor_SMD:R_0805_2012Metric, symbol Device:R_Small
- removed U6: AMS1117-3.3, Package_TO_SOT_SMD:SOT-223-3_TabPin2, symbol pak_breakout:AMS1117-3.3
- removed U7: AMS1117-5.0, Package_TO_SOT_SMD:SOT-223-3_TabPin2, symbol pak_breakout:AMS1117-5.0
- removed U8: ETA6002, Package_SO:SOIC-8-1EP_3.9x4.9mm_P1.27mm_EP2.514x3.2mm, symbol pak_breakout:ETA6002
- added BT1: Battery_Cell, Battery:BatteryHolder_Keystone_1042_1x18650, symbol Device:Battery_Cell
- added C10, C17: 100nF, Capacitor_SMD:C_0805_2012Metric, symbol Device:C_Small
- added C19: 1uF, Capacitor_SMD:C_1206_3216Metric_Pad1.42x1.75mm_HandSolder, symbol Device:C_Small
- added C21: 22uF, Capacitor_SMD:C_1206_3216Metric_Pad1.42x1.75mm_HandSolder, symbol Device:C_Small
- added C22, C8: 10uF, Capacitor_SMD:C_1206_3216Metric_Pad1.42x1.75mm_HandSolder, symbol Device:C_Small
- added D2: LED, LED_SMD:LED_0805_2012Metric_Pad1.15x1.40mm_HandSolder, symbol Device:LED
- added J6: Barrel_Jack, Connector_BarrelJack:BarrelJack_Horizontal, symbol Connector:Barrel_Jack
- added J8: Connector_USB_B_Micro, Connector_USB:USB_Micro-B_GCT_USB3076-30-A, symbol cq1re1-cache:Connector_USB_B_Micro
- added JP8: Jumper_NO_Small, Jumper:SolderJumper-2_P1.3mm_Open_RoundedPad1.0x1.5mm, symbol Device:Jumper_NO_Small
- added L2: 2.2uH, Inductor_SMD:L_Coilcraft_LPS5030, symbol Device:L
- added R12: 2k2, Resistor_SMD:R_0805_2012Metric, symbol Device:R_Small
- added R15: 500R, Resistor_SMD:R_0805_2012Metric, symbol Device:R_Small
- added U10: AMS1117-5.0, Package_TO_SOT_SMD:SOT-223-3_TabPin2, symbol pak_breakout:AMS1117-5.0
- added U5: AMS1117-3.3, Package_TO_SOT_SMD:SOT-223-3_TabPin2, symbol pak_breakout:AMS1117-3.3
- added U9: ETA6002, Package_SO:SOIC-8-1EP_3.9x4.9mm_P1.27mm_EP2.514x3.2mm, symbol pak_breakout:ETA6002
- renumbered C11 to C18, C14 to C20, C12 to C7, DCDC1 to DCDC2, JP7 to JP9
Connections:
- net ESP_3V3: now also C17.1, U5.2 (VO)
- net GND: now also BT1.2 (-), C10.2, C17.2, C19.2, C21.2, C22.2, C8.2, J6.2, J8.5 (GND), R15.2, U10.1 (GND), U5.1 (GND), U9.2 (PGND), U9.3 (NTC), U9.9 (AGND)
- net VREG: now also D2.2 (A), JP8.1, U5.3 (VI)
- net at C20.1: now also C22.1, U10.2 (VO), U9.5 (IN)
- net at C18.1, DCDC2.2 (VOUT): now also U10.3 (VI)
- net at DCDC2.1 (VIN): now also C10.1, C8.1, J6.1
- net at JP9.2: now also J8.1 (VBUS)
- new net: L2.1, U9.1 (SW)
- new net: R12.1, U9.4 (STAT)
- new net: C21.1, JP8.2, L2.2, U9.6 (SYS)
- new net: BT1.1 (+), C19.1, U9.7 (BATT)
- new net: R15.1, U9.8 (ISET)
- new net: D2.1 (K), R12.2
