File: pcbs/pcb_using_pico/psion-org2-bluetooth-adapter/x1.sch (KiCad schematic (older format))
At the start: 24 parts, among them J1 Conn_02x08_Odd_Even, J5 Conn_01x04_Female, J7 Conn_01x03_Female, M2 Si2301, U1 74LS245, U2 74LS245, U3 Pico

Commit message: Merged erroneous changes to V1.0 archive started
Parts:
- removed D1: D_Schottky, Diode_SMD:D_SOD-123, symbol Device:D_Schottky
- removed M2: Si2301, Package_TO_SOT_SMD:SOT-23, symbol cq1re1-cache:GeekAmmo_P-CHANNEL-MOSFET
- removed R10, R11, R7, R8, R9: R_Small, Resistor_SMD:R_0805_2012Metric, symbol Device:R_Small
- removed TR2: si2302, Package_TO_SOT_SMD:SOT-23, symbol cq1re1-cache:New_Library_Si2302CDS-n-channel
- removed TR3: Si2302, Package_TO_SOT_SMD:SOT-23, symbol cq1re1-cache:New_Library_Si2302CDS-n-channel
- added D3: D_Schottky, Diode_SMD:D_SOD-123, symbol Device:D_Schottky
- added R19, R20: R_Small, Resistor_SMD:R_0805_2012Metric, symbol Device:R_Small
Connections:
- net GND: now also R20.2
- net VREG: now also D3.2 (A), R19.1
- net at U3.31 (GPIO26_ADC0): now also R19.2, R20.1
- net at U3.39 (VSYS): now also D3.1 (K)
- net TRI_TX: no longer names the net of U3.21 (GPIO16)
- net TX_TO_PSION: no longer names the net of U3.24 (GPIO18)
Other:
- note added: "Pico USB could be used as USB \nserial if a connection is made to it."
